Commit message: Add complete 6-DOF URDF model, RViz config, and updated launch file

File: src/erk_description/urdf/erk.xacro (robot description, xacro)
@@ -8,5 +8,5 @@
     <origin xyz="0 0 0" rpy="0 0 0"/>
   </joint>
-  <!-- Base Link -->
+  <!-- 1. Base Link -->
   <link name="base_link">
     <visual>
@@ -29,5 +29,5 @@
     </inertial>
   </link>
-  <!-- Joint 1: Base Rotation (Revolute around Z) -->
+  <!-- Joint 1: Base Rotation (Z-axis) -->
   <joint name="Revolute_1" type="revolute">
     <parent link="base_link"/>
@@ -37,5 +37,5 @@
     <limit lower="0.0" upper="3.14159" effort="40.0" velocity="0.2"/>
   </joint>
-  <!-- Rotating Base Upper -->
+  <!-- 2. Rotating Base Upper -->
   <link name="base_link_upper">
     <visual>
@@ -58,5 +58,5 @@
     </inertial>
   </link>
-  <!-- Joint 2: Shoulder Lift (Revolute around Y) -->
+  <!-- Joint 2: Shoulder Lift (Y-axis) -->
   <joint name="Revolute_2" type="revolute">
     <parent link="base_link_upper"/>
@@ -66,5 +66,5 @@
     <limit lower="-3.14159" upper="0.0" effort="40.0" velocity="0.2"/>
   </joint>
-  <!-- Upper Arm Link 1 -->
+  <!-- 3. Upper Arm Link 1 -->
   <link name="arm_link_1">
     <visual>
@@ -87,3 +87,119 @@
     </inertial>
   </link>
+  <!-- Joint 3: Elbow Pitch (Y-axis) -->
+  <joint name="Revolute_3" type="revolute">
+    <parent link="arm_link_1"/>
+    <child link="arm_link_2"/>
+    <origin xyz="0 0 0.11312" rpy="0 0 0"/>
+    <axis xyz="0 1 0"/>
+    <limit lower="0.0" upper="3.14159" effort="40.0" velocity="0.2"/>
+  </joint>
+  <!-- 4. Forearm Link 2 -->
+  <link name="arm_link_2">
+    <visual>
+      <origin xyz="0 0 0.0491" rpy="0 0 0"/>
+      <geometry>
+        <box size="0.025 0.025 0.0982"/>
+      </geometry>
+      <material name="orange"/>
+    </visual>
+    <collision>
+      <origin xyz="0 0 0.0491" rpy="0 0 0"/>
+      <geometry>
+        <box size="0.025 0.025 0.0982"/>
+      </geometry>
+    </collision>
+    <inertial>
+      <mass value="0.1"/>
+      <origin xyz="0 0 0.0491"/>
+      <inertia ixx="0.0001" ixy="0" ixz="0" iyy="0.0001" iyz="0" izz="0.0001"/>
+    </inertial>
+  </link>
+  <!-- Joint 4: Forearm Roll (Z-axis) -->
+  <joint name="Revolute_4" type="revolute">
+    <parent link="arm_link_2"/>
+    <child link="arm_link_3"/>
+    <origin xyz="0 0 0.0982" rpy="0 0 0"/>
+    <axis xyz="0 0 1"/>
+    <limit lower="-1.5708" upper="1.5708" effort="20.0" velocity="0.2"/>
+  </joint>
+  <!-- 5. Wrist Bracket Link 3 -->
+  <link name="arm_link_3">
+    <visual>
+      <origin xyz="0 0 0.016" rpy="0 0 0"/>
+      <geometry>
+        <box size="0.02 0.02 0.0321"/>
+      </geometry>
+      <material name="white"/>
+    </visual>
+    <collision>
+      <origin xyz="0 0 0.016" rpy="0 0 0"/>
+      <geometry>
+        <box size="0.02 0.02 0.0321"/>
+      </geometry>
+    </collision>
+    <inertial>
+      <mass value="0.05"/>
+      <origin xyz="0 0 0.016"/>
+      <inertia ixx="0.00005" ixy="0" ixz="0" iyy="0.00005" iyz="0" izz="0.00005"/>
+    </inertial>
+  </link>
+  <!-- Joint 5: Wrist Tilt (Y-axis) -->
+  <joint name="Revolute_5" type="revolute">
+    <parent link="arm_link_3"/>
+    <child link="gripper_base"/>
+    <origin xyz="0 0 0.0321" rpy="0 0 0"/>
+    <axis xyz="0 1 0"/>
+    <limit lower="-1.5708" upper="1.5708" effort="20.0" velocity="0.2"/>
+  </joint>
+  <!-- 6. Gripper Base -->
+  <link name="gripper_base">
+    <visual>
+      <origin xyz="0 0 0.015" rpy="0 0 0"/>
+      <geometry>
+        <box size="0.04 0.02 0.03"/>
+      </geometry>
+      <material name="orange"/>
+    </visual>
+    <collision>
+      <origin xyz="0 0 0.015" rpy="0 0 0"/>
+      <geometry>
+        <box size="0.04 0.02 0.03"/>
+      </geometry>
+    </collision>
+    <inertial>
+      <mass value="0.05"/>
+      <origin xyz="0 0 0.015"/>
+      <inertia ixx="0.00005" ixy="0" ixz="0" iyy="0.00005" iyz="0" izz="0.00005"/>
+    </inertial>
+  </link>
+  <!-- Joint 6: Gripper Jaw (Revolute/Prismatic) -->
+  <joint name="Gripper" type="revolute">
+    <parent link="gripper_base"/>
+    <child link="gripper_finger_left"/>
+    <origin xyz="0.015 0 0.03" rpy="0 0 0"/>
+    <axis xyz="0 1 0"/>
+    <limit lower="0.0" upper="0.8" effort="10.0" velocity="0.2"/>
+  </joint>
+  <!-- Left Finger Link -->
+  <link name="gripper_finger_left">
+    <visual>
+      <origin xyz="0 0 0.015" rpy="0 0 0"/>
+      <geometry>
+        <box size="0.005 0.01 0.03"/>
+      </geometry>
+      <material name="white"/>
+    </visual>
+    <collision>
+      <origin xyz="0 0 0.015" rpy="0 0 0"/>
+      <geometry>
+        <box size="0.005 0.01 0.03"/>
+      </geometry>
+    </collision>
+    <inertial>
+      <mass value="0.01"/>
+      <origin xyz="0 0 0.015"/>
+      <inertia ixx="0.00001" ixy="0" ixz="0" iyy="0.00001" iyz="0" izz="0.00001"/>
+    </inertial>
+  </link>
 </robot>

Commit message: Add Gazebo physics simulation, ros2_control configuration, and gazebo launch file

File: src/erk_description/urdf/erk.xacro (robot description, xacro)
@@ -203,3 +203,45 @@
     </inertial>
   </link>
+  <!-- Gazebo Simulation Plugin -->
+  <gazebo>
+    <plugin filename="gz_ros2_control-system" name="gz_ros2_control::GazeboSimROS2ControlPlugin">
+      <parameters>$(find erk_description)/config/gazebo_controllers.yaml</parameters>
+    </plugin>
+  </gazebo>
+  <!-- ros2_control Hardware Interface Definition -->
+  <ros2_control name="GazeboSystem" type="system">
+    <hardware>
+      <plugin>gz_ros2_control/GazeboSimSystem</plugin>
+    </hardware>
+    <joint name="Revolute_1">
+      <command_interface name="position"/>
+      <state_interface name="position"/>
+      <state_interface name="velocity"/>
+    </joint>
+    <joint name="Revolute_2">
+      <command_interface name="position"/>
+      <state_interface name="position"/>
+      <state_interface name="velocity"/>
+    </joint>
+    <joint name="Revolute_3">
+      <command_interface name="position"/>
+      <state_interface name="position"/>
+      <state_interface name="velocity"/>
+    </joint>
+    <joint name="Revolute_4">
+      <command_interface name="position"/>
+      <state_interface name="position"/>
+      <state_interface name="velocity"/>
+    </joint>
+    <joint name="Revolute_5">
+      <command_interface name="position"/>
+      <state_interface name="position"/>
+      <state_interface name="velocity"/>
+    </joint>
+    <joint name="Gripper">
+      <command_interface name="position"/>
+      <state_interface name="position"/>
+      <state_interface name="velocity"/>
+    </joint>
+  </ros2_control>
 </robot>
